Commit message: UPDATE: change color and naming

File: assets/urdf/cartpole.urdf (robot description, URDF)
Before this commit: robot physics, 3 links, 2 joints
Links:
- removed link slideBar
- added link slide_bar, mass 0; visual box size=30 0.05 0.05
Joints:
- joint slider_to_cart: parent slideBar -> slide_bar
